Commit message: increased mass to stabilize robot and added some comments in the urdfs

File: niryo_one_description/urdf/v2/gripper/niryo_gripper_2.urdf.xacro (robot description, xacro)
@@ -7,4 +7,6 @@
       <inertia ixx="${m*(3*r*r+h*h)/12}" ixy = "0" ixz = "0" iyy="${m*(3*r*r+h*h)/12}" iyz = "0" izz="${m*r*r/2}" />
    </xacro:macro>
+    <!-- The gripper needs to be fixed -->
+    <!-- Should add gripper and transmission tags to gripper joints -->
    <xacro:macro name="default_transmission" params="jname">
     <transmission name="${jname}_trans">

File: niryo_one_description/urdf/v2/niryo_one.urdf (robot description, URDF)
Before this commit: robot niryo_one, 16 links, 15 joints
Links:
- link base_link: mass 2 -> 5

File: niryo_one_description/urdf/v2/niryo_one.urdf.xacro (robot description, xacro)
@@ -63,10 +63,16 @@
         <inertial>
       		<origin xyz="0 0 0" rpy="0 0 0"/>
-      		<mass value="2"/>
+      		<mass value="100"/>
 			<!--to change-->
-      		<inertia
-        		ixx="0.0" ixy="0.0" ixz="0.0"
-        		iyy="0.0" iyz="0.0"
-        		izz="0.0"/>
+      <!-- This 100 kg value is too much but at least it stabilizes the robot well enough -->
+      <!-- the other links of the arm were considered solid lines and the inertias were calculated according
+           to the link bellow:
+           https://en.wikipedia.org/wiki/List_of_moments_of_inertia#List_of_3D_inertia_tensors -->
+           <!-- The robot is not always super stable but at least it seems to work -->
+           <!-- Maybe also the center of mass has to be fixed -->
+      		<inertia
+        		ixx="0.21666" ixy="0.0" ixz="0.0"
+        		iyy="0.32666" iyz="0.0"
+        		izz="0.21666"/>
     	</inertial>
 	</link>
@@ -86,75 +92,75 @@
         <inertial>
       		<origin xyz="0 0 0" rpy="0 0 0"/>
-      		<mass value="1"/>
-      		<inertia
-        		ixx="1.0" ixy="0.0" ixz="0.0"
+      		<mass value="0.4"/>
+      		<inertia
+        		ixx="0.00221" ixy="0.0" ixz="0.0"
+        		iyy="0.0" iyz="0.0"
+        		izz="0.00221"/>
+    	</inertial>
+	</link>
+    <link name="arm_link">
+		<visual>
+			<origin xyz="0 0 0" rpy="0 0 0" />
+			<geometry>
+                <mesh filename="package://niryo_one_description/meshes/v2/collada/arm_link.dae" />
+			</geometry>
+		</visual>
+        <collision>
+			<origin xyz="0 0 0" rpy="0 0 0" />
+            <geometry>
+                <mesh filename="package://niryo_one_description/meshes/v2/stl/arm_link.stl" />
+            </geometry>
+        </collision>
+        <inertial>
+      		<origin xyz="0 0 0" rpy="0 0 0"/>
+      		<mass value="0.4"/>
+      		<inertia
+        		ixx="0.0022" ixy="0.0" ixz="0.0"
+        		iyy="0.0" iyz="0.0"
+        		izz="0.0022"/>
+    	</inertial>
+	</link>
+    <link name="elbow_link">
+		<visual>
+			<origin xyz="0 0 0" rpy="0 0 0" />
+			<geometry>
+                <mesh filename="package://niryo_one_description/meshes/v2/collada/elbow_link.dae" />
+			</geometry>
+		</visual>
+        <collision>
+			<origin xyz="0 0 0" rpy="0 0 0" />
+            <geometry>
+                <mesh filename="package://niryo_one_description/meshes/v2/stl/elbow_link.stl" />
+            </geometry>
+        </collision>
+        <inertial>
+      		<origin xyz="0 0 0" rpy="0 0 0"/>
+      		<mass value="0.4"/>
+      		<inertia
+        		ixx="0.0022" ixy="0.0" ixz="0.0"
+        		iyy="0.0" iyz="0.0"
+        		izz="0.022"/>
+    	</inertial>
+	</link>
+    <link name="forearm_link">
+		<visual>
+			<origin xyz="0 0 0" rpy="0 0 0" />
+			<geometry>
+                <mesh filename="package://niryo_one_description/meshes/v2/collada/forearm_link.dae" />
+			</geometry>
+		</visual>
+        <collision>
+			<origin xyz="0 0 0" rpy="0 0 0" />
+            <geometry>
+                <mesh filename="package://niryo_one_description/meshes/v2/stl/forearm_link.stl" />
+            </geometry>
+        </collision>
+        <inertial>
+      		<origin xyz="0 0 0" rpy="0 0 0"/>
+      		<mass value="0.4"/>
+      		<inertia
+        		ixx="0.0022" ixy="0.0" ixz="0.0"
         		iyy="1.0" iyz="0.0"
-        		izz="1.0"/>
-    	</inertial>
-	</link>
-    <link name="arm_link">
-		<visual>
-			<origin xyz="0 0 0" rpy="0 0 0" />
-			<geometry>
-                <mesh filename="package://niryo_one_description/meshes/v2/collada/arm_link.dae" />
-			</geometry>
-		</visual>
-        <collision>
-			<origin xyz="0 0 0" rpy="0 0 0" />
-            <geometry>
-                <mesh filename="package://niryo_one_description/meshes/v2/stl/arm_link.stl" />
-            </geometry>
-        </collision>
-        <inertial>
-      		<origin xyz="0 0 0" rpy="0 0 0"/>
-      		<mass value="0.5"/>
-      		<inertia
-        		ixx="1.0" ixy="0.0" ixz="0.0"
-        		iyy="1.0" iyz="0.0"
-        		izz="1.0"/>
-    	</inertial>
-	</link>
-    <link name="elbow_link">
-		<visual>
-			<origin xyz="0 0 0" rpy="0 0 0" />
-			<geometry>
-                <mesh filename="package://niryo_one_description/meshes/v2/collada/elbow_link.dae" />
-			</geometry>
-		</visual>
-        <collision>
-			<origin xyz="0 0 0" rpy="0 0 0" />
-            <geometry>
-                <mesh filename="package://niryo_one_description/meshes/v2/stl/elbow_link.stl" />
-            </geometry>
-        </collision>
-        <inertial>
-      		<origin xyz="0 0 0" rpy="0 0 0"/>
-      		<mass value="0.4"/>
-      		<inertia
-        		ixx="1.0" ixy="0.0" ixz="0.0"
-        		iyy="1.0" iyz="0.0"
-        		izz="1.0"/>
-    	</inertial>
-	</link>
-    <link name="forearm_link">
-		<visual>
-			<origin xyz="0 0 0" rpy="0 0 0" />
-			<geometry>
-                <mesh filename="package://niryo_one_description/meshes/v2/collada/forearm_link.dae" />
-			</geometry>
-		</visual>
-        <collision>
-			<origin xyz="0 0 0" rpy="0 0 0" />
-            <geometry>
-                <mesh filename="package://niryo_one_description/meshes/v2/stl/forearm_link.stl" />
-            </geometry>
-        </collision>
-        <inertial>
-      		<origin xyz="0 0 0" rpy="0 0 0"/>
-      		<mass value="0.3"/>
-      		<inertia
-        		ixx="1.0" ixy="0.0" ixz="0.0"
-        		iyy="1.0" iyz="0.0"
-        		izz="1.0"/>
+        		izz="0.0022"/>
     	</inertial>
 	</link>
@@ -176,7 +182,7 @@
       		<mass value="0.2"/>
       		<inertia
-        		ixx="1.0" ixy="0.0" ixz="0.0"
-        		iyy="1.0" iyz="0.0"
-        		izz="1.0"/>
+        		ixx="0.0011" ixy="0.0" ixz="0.0"
+        		iyy="0.0" iyz="0.0"
+        		izz="0.0011"/>
     	</inertial>
 	</link>

Commit message: made mimic joint work in gazebo

File: niryo_one_description/urdf/v2/gripper/niryo_gripper_2.urdf.xacro (robot description, xacro)
@@ -4,4 +4,6 @@
    xmlns:interface="http://playerstage.sourceforge.net/gazebo/xmlschema/#interface"
    xmlns:xacro="http://ros.org/wiki/xacro" name="egp_40">
+<!-- Dependency!! -->
+<!-- https://github.com/roboticsgroup/roboticsgroup_gazebo_plugins -->
    <xacro:macro name="cylinder_inertia" params="m r h">
       <inertia ixx="${m*(3*r*r+h*h)/12}" ixy = "0" ixz = "0" iyy="${m*(3*r*r+h*h)/12}" iyz = "0" izz="${m*r*r/2}" />
@@ -34,4 +36,5 @@
             <origin xyz="0 0 0" />
             <cylinder_inertia m="0.20" r="0.05" h="0.05" />
+            <gravity>1</gravity>
          </inertial>
          <visual>
@@ -53,5 +56,5 @@
       <gazebo reference="${prefix}base_link">
          <material>Gazebo/Black</material>
-         <turnGravityOff>false</turnGravityOff>
+         <!--turnGravityOff>false</turnGravityOff-->
       </gazebo>
       <!-- GEAR LEFT LINK -->
@@ -59,5 +62,5 @@
          <parent link="${prefix}base_link"/>
          <child link="${prefix}gear_left_link"/>
-            <origin xyz="0.016 0 0.005" rpy="0 0 0" />
+            <origin xyz="0.016 0.0 0.005" rpy="0 0 0" />
          <axis xyz="0 -1 0" />
  	 <limit effort="1000.0" lower="-1.2" upper="0.0" velocity="0.5"/>
@@ -66,4 +69,5 @@
         <implicitSpringDamper>1</implicitSpringDamper>
       </gazebo>
+      <!-- gripper gear left link -->
       <link name="${prefix}gear_left_link">
          <inertial>
@@ -71,4 +75,5 @@
             <origin xyz="0 0 0" />
             <cylinder_inertia m="0.20" r="0.05" h="0.05" />
+            <gravity>1</gravity>
          </inertial>
          <visual>
@@ -99,4 +104,5 @@
         <implicitSpringDamper>1</implicitSpringDamper>
       </gazebo>
+      <!-- gripper gear right link -->
       <link name="${prefix}gear_right_link">
          <inertial>
@@ -104,4 +110,5 @@
             <origin xyz="0 0 0" />
             <cylinder_inertia m="0.20" r="0.05" h="0.05" />
+            <gravity>1</gravity>
          </inertial>
          <visual>
@@ -115,5 +122,5 @@
          </visual>
          <collision>
-            <origin xyz="0.0 0 0" rpy="0 0 0" />
+            <origin xyz="0.0 0.0 0.0" rpy="0 0 0" />
             <geometry>
                <mesh filename="package://niryo_one_description/meshes/v2/stl/G2_GearRight.STL" scale="0.001 0.001 0.001"/>
@@ -133,4 +140,5 @@
         <implicitSpringDamper>1</implicitSpringDamper>
       </gazebo>
+      <!-- left finger base link -->
       <link name="${prefix}left_finger_base_link">
          <inertial>
@@ -138,4 +146,5 @@
             <origin xyz="0 0 0" />
             <cylinder_inertia m="0.02" r="0.01" h="0.01" />
+            <gravity>1</gravity>
          </inertial>
          <visual>
@@ -149,5 +158,5 @@
          </visual>
          <collision>
-            <origin xyz="0.0 0 0" rpy="0 0 0" />
+            <origin xyz="0.0 0.0 0.0" rpy="0 0 0" />
             <geometry>
                <mesh filename="package://niryo_one_description/meshes/v2/stl/G2_Clamp.STL" scale="0.001 0.001 0.001"/>
@@ -167,4 +176,5 @@
         <implicitSpringDamper>1</implicitSpringDamper>
       </gazebo>
+      <!-- right finger base link -->
       <link name="${prefix}right_finger_base_link">
          <inertial>
@@ -172,4 +182,5 @@
             <origin xyz="0 0 0" />
             <cylinder_inertia m="0.02" r="0.01" h="0.01" />
+            <gravity>1</gravity>
          </inertial>
          <visual>
@@ -193,12 +204,13 @@
          <parent link="${prefix}base_link"/>
          <child link="${prefix}rod_left_link"/>
-            <origin xyz="0.014 0 0.027" rpy="0 0 0" />
+            <origin xyz="0.014 0.0 0.027" rpy="0 0 0" />
         <axis xyz="0 -1 0" />
  	 <limit effort="1000.0" lower="-1.2" upper="1.2" velocity="0.5"/>
-	<mimic joint="${prefix}gear_left_joint" multiplier="1" offset="0.0"/>
+	<mimic joint="${prefix}gear_left_joint" multiplier="1" offset="0"/>
       </joint>
        <gazebo reference="${prefix}rod_left_joint">
         <implicitSpringDamper>1</implicitSpringDamper>
       </gazebo>
+      <!-- rod left link -->
       <link name="${prefix}rod_left_link">
          <inertial>
@@ -206,4 +218,5 @@
             <origin xyz="0 0 0" />
             <cylinder_inertia m="0.20" r="0.05" h="0.05" />
+            <gravity>1</gravity>
          </inertial>
          <visual>
@@ -217,5 +230,5 @@
          </visual>
          <collision>
-            <origin xyz="0.0 0 0" rpy="0 0 0" />
+            <origin xyz="0.0 0.0 0.0" rpy="0 0 0" />
             <geometry>
                <mesh filename="package://niryo_one_description/meshes/v2/stl/G2_Rod.STL" scale="0.001 0.001 0.001"/>
@@ -227,5 +240,5 @@
          <parent link="${prefix}base_link"/>
          <child link="${prefix}rod_right_link"/>
-            <origin xyz="0.0 0 0.027" rpy="0 0 0" />
+            <origin xyz="0.0 0.0 0.027" rpy="0 0 0" />
          <axis xyz="0 -1 0" />
  	 <limit effort="1000.0" lower="-1.2" upper="1.2" velocity="0.5"/>
@@ -235,4 +248,5 @@
         <implicitSpringDamper>1</implicitSpringDamper>
       </gazebo>
+      <!-- rod right link -->
       <link name="${prefix}rod_right_link">
          <inertial>
@@ -240,4 +254,5 @@
             <origin xyz="0 0 0" />
             <cylinder_inertia m="0.20" r="0.05" h="0.05" />
+            <gravity>1</gravity>
          </inertial>
          <visual>
@@ -251,5 +266,5 @@
          </visual>
          <collision>
-            <origin xyz="0.0 0 0" rpy="0 0 0" />
+            <origin xyz="0.0 0.0 0.0" rpy="0 0 0" />
             <geometry>
                <mesh filename="package://niryo_one_description/meshes/v2/stl/G2_Rod.STL" scale="0.001 0.001 0.001"/>
@@ -257,7 +272,52 @@
          </collision>
       </link>
+      <!-- GEORGE_LEFT -->
+      <!--joint name="${prefix}george_left_joint" type="revolute">
+         <parent link="${prefix}rod_left_link"/>
+         <child link="${prefix}left_finger_base_link"/>
+            <origin xyz="0.007 10 0.027" rpy="1.57 0 0" />
+        <axis xyz="0 -1 0" />
+ 	 <limit effort="1000.0" lower="-1.2" upper="1.2" velocity="0.5"/>
+      </joint-->
+       <!--gazebo reference="${prefix}george_left_joint">
+        <implicitSpringDamper>1</implicitSpringDamper>
+      </gazebo-->
+      <!-- george left link -->
+      <!--link name="${prefix}george_left_link">
+         <inertial>
+            <mass value="0.25" />
+            <origin xyz="0 0 0" />
+            <cylinder_inertia m="0.20" r="0.05" h="0.05" />
+         </inertial>
+         <visual>
+	<origin xyz="0.027 0.02 0.008" rpy="0.0 0.0 3.14" />
+            <geometry>
+               <mesh filename="package://niryo_one_description/meshes/v2/stl/G2_George.STL" scale="0.001 0.001 0.001"/>
+            </geometry>
+            <material name="black">
+  		<color rgba="0.0 0.0 0.0 1.0"/>
+            </material>
+         </visual>
+         <collision>
+            <origin xyz="0.0 0.0 0.0" rpy="0 0 0" />
+            <geometry>
+               <mesh filename="package://niryo_one_description/meshes/v2/stl/G2_George.STL" scale="0.001 0.001 0.001"/>
+            </geometry>
+         </collision>
+      </link-->
+      <!-- GEORGE RIGHT -->
+      <!--joint name="${prefix}george_right_joint" type="revolute">
+         <parent link="${prefix}rod_right_link"/>
+         <child link="${prefix}right_finger_base_link"/>
+            <origin xyz="-0.007 0.0 0.027" rpy="0 0 0" />
+        <axis xyz="0 -1 0" />
+ 	 <limit effort="1000.0" lower="-1.2" upper="1.2" velocity="0.5"/>
+      </joint-->
+       <!--gazebo reference="${prefix}george_right_joint">
+        <implicitSpringDamper>1</implicitSpringDamper>
+      </gazebo-->
     <!-- Mimic joints -->
     <gazebo>
-      <plugin filename="libgazebo_mimic_joint_plugin.so" name="${prefix}mimic_gripper2_1">
+      <plugin filename="libroboticsgroup_gazebo_mimic_joint_plugin.so" name="${prefix}mimic_gripper2_1">
         <joint>${prefix}gear_left_joint</joint>
         <mimicJoint>${prefix}rod_left_joint</mimicJoint>
@@ -265,5 +325,5 @@
         <offset>0.0</offset>
       </plugin>
-      <plugin filename="libgazebo_mimic_joint_plugin.so" name="${prefix}mimic_gripper2_2">
+      <plugin filename="libroboticsgroup_gazebo_mimic_joint_plugin.so" name="${prefix}mimic_gripper2_2">
         <joint>${prefix}gear_right_joint</joint>
         <mimicJoint>${prefix}rod_right_joint</mimicJoint>
@@ -271,5 +331,5 @@
         <offset>0.0</offset>
       </plugin>
-      <plugin filename="libgazebo_mimic_joint_plugin.so" name="${prefix}mimic_gripper2_3">
+      <plugin filename="libroboticsgroup_gazebo_mimic_joint_plugin.so" name="${prefix}mimic_gripper2_3">
         <joint>${prefix}gear_left_joint</joint>
         <mimicJoint>${prefix}left_finger_base_joint</mimicJoint>
@@ -277,5 +337,5 @@
         <offset>0</offset>
       </plugin>
-      <plugin filename="libgazebo_mimic_joint_plugin.so" name="${prefix}mimic_gripper2_4">
+      <plugin filename="libroboticsgroup_gazebo_mimic_joint_plugin.so" name="${prefix}mimic_gripper2_4">
         <joint>${prefix}gear_right_joint</joint>
         <mimicJoint>${prefix}right_finger_base_joint</mimicJoint>

File: niryo_one_description/urdf/v2/niryo_one.urdf (robot description, URDF)
Before this commit: robot niryo_one, 16 links, 15 joints
Links:
- link arm_link: mass 0.5 -> 0.4
- link base_link: mass 5 -> 100
- link forearm_link: mass 0.3 -> 0.4
- link shoulder_link: mass 1 -> 0.4
Joints:
- joint gripper_gear_left_joint: origin xyz=0.016 0 0.005 rpy=0 0 0 -> xyz=0.016 0.0 0.005 rpy=0 0 0
- joint gripper_rod_left_joint: mimic joint=gripper_gear_left_joint multiplier=1 offset=0.0 -> joint=gripper_gear_left_joint multiplier=1 offset=0; origin xyz=0.014 0 0.027 rpy=0 0 0 -> xyz=0.014 0.0 0.027 rpy=0 0 0
- joint gripper_rod_right_joint: origin xyz=0.0 0 0.027 rpy=0 0 0 -> xyz=0.0 0.0 0.027 rpy=0 0 0

Commit message: changed the rpy of rod joints

File: niryo_one_description/urdf/v2/gripper/niryo_gripper_2.urdf.xacro (robot description, xacro)
@@ -204,5 +204,5 @@
          <parent link="${prefix}base_link"/>
          <child link="${prefix}rod_left_link"/>
-            <origin xyz="0.014 0.0 0.027" rpy="0 0 0" />
+         <origin xyz="0.014 0.0 0.027" rpy="0 0.261799 0" />  <!-- 0.261799 is 15 degrees -->
         <axis xyz="0 -1 0" />
  	 <limit effort="1000.0" lower="-1.2" upper="1.2" velocity="0.5"/>
@@ -240,5 +240,5 @@
          <parent link="${prefix}base_link"/>
          <child link="${prefix}rod_right_link"/>
-            <origin xyz="0.0 0.0 0.027" rpy="0 0 0" />
+          <origin xyz="0.0 0.0 0.027" rpy="0 -0.261799 0" /> <!-- -0.261799 is 15 degrees -->
          <axis xyz="0 -1 0" />
  	 <limit effort="1000.0" lower="-1.2" upper="1.2" velocity="0.5"/>
