Commit message: might have managed to fix the flying of the clamps

File: niryo_one_description/urdf/v2/gripper/niryo_gripper_2.urdf.xacro (robot description, xacro)
@@ -16,6 +16,6 @@
       <joint name="${jname}_joint">
         <hardwareInterface>hardware_interface/EffortJointInterface</hardwareInterface>
-        <!--<hardwareInterface>hardware_interface/PositionJointInterface</hardwareInterface>
-        <hardwareInterface>hardware_interface/VelocityJointInterface</hardwareInterface>-->
+        <!--hardwareInterface>hardware_interface/PositionJointInterface</hardwareInterface-->
+        <!--hardwareInterface>hardware_interface/VelocityJointInterface</hardwareInterface-->
       </joint>
       <actuator name="${jname}_motor">
@@ -64,5 +64,5 @@
             <origin xyz="0.016 0.0 0.005" rpy="0 0 0" />
          <axis xyz="0 -1 0" />
- 	 <limit effort="1000.0" lower="-1.2" upper="0.0" velocity="0.5"/>
+ 	       <limit effort="1000.0" lower="-1.2" upper="0.0" velocity="0.5"/>
       </joint>
       <gazebo reference="${prefix}gear_left_joint">
@@ -113,5 +113,5 @@
          </inertial>
          <visual>
-            <origin xyz="-0.008 0.02 0.045" rpy=" 3.14 0  0 " />
+            <origin xyz="-0.008 0.02 0.045" rpy="3.14 0  0" />
             <geometry>
                <mesh filename="package://niryo_one_description/meshes/v2/stl/G2_GearRight.STL" scale="0.001 0.001 0.001"/>
@@ -132,8 +132,15 @@
          <parent link="${prefix}gear_left_link"/>
          <child link="${prefix}left_finger_base_link"/>
-            <origin xyz="0.01 0.0 0.035" rpy="0 0 0" />
+         <origin xyz="0.01 0.0 0.035" rpy="0 -0.0174533 0" />
          <axis xyz="0 -1 0" />
- 	 <limit effort="1000.0" lower="-1.2" upper="1.2" velocity="0.5"/>
-	<mimic joint="${prefix}gear_left_joint" multiplier="-1" offset="0"/>
+				 <dynamics damping="0.7"/>
+         <gazebo>
+      		<stopErp>0.2</stopErp>
+      		<stopCfm>0.0</stopCfm>
+    		</gazebo>
+ 	      <limit effort="1000.0" lower="-1.2" upper="1.2" velocity="0.5">
+          <gazebo/>
+        </limit>
+	      <mimic joint="${prefix}gear_left_joint" multiplier="-1" offset="0"/>
       </joint>
       <gazebo reference="${prefix}left_finger_base_joint">
@@ -166,10 +173,17 @@
       <!-- GRIPPER CLAMP RIGHT -->
       <joint name="${prefix}right_finger_base_joint" type="revolute">
-         <parent link="${prefix}gear_right_link"/>
-         <child link="${prefix}right_finger_base_link"/>
-         <origin xyz="-0.01 0.0 0.035" rpy=" 0 0 0" />
-         <axis xyz="0 -1 0" />
- 	 <limit effort="1000.0" lower="-1.2" upper="1.2" velocity="0.5"/>
-	<mimic joint="${prefix}gear_right_joint" multiplier="-1" offset="0"/>
+        <parent link="${prefix}gear_right_link"/>
+        <child link="${prefix}right_finger_base_link"/>
+        <origin xyz="-0.01 0.0 0.035" rpy=" 0 0.0174533 0" />
+        <axis xyz="0 -1 0" />
+			  <dynamics damping="0.7"/>
+		 	  <gazebo>
+      	  <stopErp>0.2</stopErp>
+      	  <stopCfm>0.0</stopCfm>
+    	  </gazebo>
+ 	      <limit effort="1000.0" lower="-1.2" upper="1.2" velocity="0.5">
+          <gazebo/>
+        </limit>
+	      <mimic joint="${prefix}gear_right_joint" multiplier="-1" offset="0"/>
       </joint>
       <gazebo reference="${prefix}right_finger_base_joint">
@@ -272,49 +286,4 @@
          </collision>
       </link>
-      <!-- GEORGE_LEFT -->
-      <!--joint name="${prefix}george_left_joint" type="revolute">
-         <parent link="${prefix}rod_left_link"/>
-         <child link="${prefix}left_finger_base_link"/>
-            <origin xyz="0.007 10 0.027" rpy="1.57 0 0" />
-        <axis xyz="0 -1 0" />
- 	 <limit effort="1000.0" lower="-1.2" upper="1.2" velocity="0.5"/>
-      </joint-->
-       <!--gazebo reference="${prefix}george_left_joint">
-        <implicitSpringDamper>1</implicitSpringDamper>
-      </gazebo-->
-      <!-- george left link -->
-      <!--link name="${prefix}george_left_link">
-         <inertial>
-            <mass value="0.25" />
-            <origin xyz="0 0 0" />
-            <cylinder_inertia m="0.20" r="0.05" h="0.05" />
-         </inertial>
-         <visual>
-	<origin xyz="0.027 0.02 0.008" rpy="0.0 0.0 3.14" />
-            <geometry>
-               <mesh filename="package://niryo_one_description/meshes/v2/stl/G2_George.STL" scale="0.001 0.001 0.001"/>
-            </geometry>
-            <material name="black">
-  		<color rgba="0.0 0.0 0.0 1.0"/>
-            </material>
-         </visual>
-         <collision>
-            <origin xyz="0.0 0.0 0.0" rpy="0 0 0" />
-            <geometry>
-               <mesh filename="package://niryo_one_description/meshes/v2/stl/G2_George.STL" scale="0.001 0.001 0.001"/>
-            </geometry>
-         </collision>
-      </link-->
-      <!-- GEORGE RIGHT -->
-      <!--joint name="${prefix}george_right_joint" type="revolute">
-         <parent link="${prefix}rod_right_link"/>
-         <child link="${prefix}right_finger_base_link"/>
-            <origin xyz="-0.007 0.0 0.027" rpy="0 0 0" />
-        <axis xyz="0 -1 0" />
- 	 <limit effort="1000.0" lower="-1.2" upper="1.2" velocity="0.5"/>
-      </joint-->
-       <!--gazebo reference="${prefix}george_right_joint">
-        <implicitSpringDamper>1</implicitSpringDamper>
-      </gazebo-->
     <!-- Mimic joints -->
     <gazebo>

File: niryo_one_description/urdf/v2/niryo_one.urdf (robot description, URDF)
Before this commit: robot niryo_one, 16 links, 15 joints
Joints:
- joint gripper_left_finger_base_joint: origin xyz=0.01 0.0 0.035 rpy=0 0 0 -> xyz=0.01 0.0 0.035 rpy=0 -0.0174533 0
- joint gripper_right_finger_base_joint: origin xyz=-0.01 0.0 0.035 rpy= 0 0 0 -> xyz=-0.01 0.0 0.035 rpy= 0 0.0174533 0
- joint gripper_rod_left_joint: origin xyz=0.014 0.0 0.027 rpy=0 0 0 -> xyz=0.014 0.0 0.027 rpy=0 0.261799 0
- joint gripper_rod_right_joint: origin xyz=0.0 0.0 0.027 rpy=0 0 0 -> xyz=0.0 0.0 0.027 rpy=0 -0.261799 0

Commit message: Made also the rod joints behave well

File: niryo_one_description/urdf/v2/gripper/niryo_gripper_2.urdf.xacro (robot description, xacro)
@@ -216,10 +216,17 @@
       <!-- ROD LEFT -->
       <joint name="${prefix}rod_left_joint" type="revolute">
-         <parent link="${prefix}base_link"/>
-         <child link="${prefix}rod_left_link"/>
-         <origin xyz="0.014 0.0 0.027" rpy="0 0.261799 0" />  <!-- 0.261799 is 15 degrees -->
+        <parent link="${prefix}base_link"/>
+        <child link="${prefix}rod_left_link"/>
+        <origin xyz="0.014 0.0 0.027" rpy="0 0.261799 0" />  <!-- 0.261799 is 15 degrees -->
         <axis xyz="0 -1 0" />
- 	 <limit effort="1000.0" lower="-1.2" upper="1.2" velocity="0.5"/>
-	<mimic joint="${prefix}gear_left_joint" multiplier="1" offset="0"/>
+				<dynamics damping="0.7"/>
+        <gazebo>
+      	  <stopErp>0.2</stopErp>
+      	  <stopCfm>0.0</stopCfm>
+    	  </gazebo>
+ 	      <limit effort="1000.0" lower="-1.2" upper="1.2" velocity="0.5">
+          <gazebo/>
+        </limit>
+	      <mimic joint="${prefix}gear_left_joint" multiplier="1" offset="0"/>
       </joint>
        <gazebo reference="${prefix}rod_left_joint">
@@ -252,10 +259,17 @@
       <!-- ROD RIGHT -->
       <joint name="${prefix}rod_right_joint" type="revolute">
-         <parent link="${prefix}base_link"/>
-         <child link="${prefix}rod_right_link"/>
-          <origin xyz="0.0 0.0 0.027" rpy="0 -0.261799 0" /> <!-- -0.261799 is 15 degrees -->
-         <axis xyz="0 -1 0" />
- 	 <limit effort="1000.0" lower="-1.2" upper="1.2" velocity="0.5"/>
-	<mimic joint="${prefix}gear_right_joint" multiplier="1" offset="0.0"/>
+        <parent link="${prefix}base_link"/>
+        <child link="${prefix}rod_right_link"/>
+        <origin xyz="0.0 0.0 0.027" rpy="0 -0.261799 0" /> <!-- -0.261799 is 15 degrees -->
+        <axis xyz="0 -1 0" />
+        <dynamics damping="0.7"/>
+        <gazebo>
+      	  <stopErp>0.2</stopErp>
+      	  <stopCfm>0.0</stopCfm>
+    	  </gazebo>
+ 	      <limit effort="1000.0" lower="-1.2" upper="1.2" velocity="0.5">
+          <gazebo/>
+        </limit>
+	      <mimic joint="${prefix}gear_right_joint" multiplier="1" offset="0.0"/>
       </joint>
       <gazebo reference="${prefix}rod_right_joint">
@@ -291,12 +305,12 @@
         <joint>${prefix}gear_left_joint</joint>
         <mimicJoint>${prefix}rod_left_joint</mimicJoint>
-        <multiplier>1.0</multiplier>
-        <offset>0.0</offset>
+        <multiplier>1.186</multiplier>
+        <offset>0.261799</offset>
       </plugin>
       <plugin filename="libroboticsgroup_gazebo_mimic_joint_plugin.so" name="${prefix}mimic_gripper2_2">
         <joint>${prefix}gear_right_joint</joint>
         <mimicJoint>${prefix}rod_right_joint</mimicJoint>
-        <multiplier>1.0</multiplier>
-        <offset>0.0</offset>
+        <multiplier>1.186</multiplier>
+        <offset>-0.261799</offset>
       </plugin>
       <plugin filename="libroboticsgroup_gazebo_mimic_joint_plugin.so" name="${prefix}mimic_gripper2_3">

Commit message: added some comments and a cube in the simulation

File: niryo_one_description/urdf/v2/gripper/niryo_gripper_2.urdf.xacro (robot description, xacro)
@@ -165,5 +165,5 @@
          </visual>
          <collision>
-            <origin xyz="0.0 0.0 0.0" rpy="0 0 0" />
+            <origin xyz="0.0 0.0 0.2" rpy="0 0 0" />
             <geometry>
                <mesh filename="package://niryo_one_description/meshes/v2/stl/G2_Clamp.STL" scale="0.001 0.001 0.001"/>
@@ -208,5 +208,5 @@
          </visual>
          <collision>
-            <origin xyz="0.0 0 0" rpy="0 0 0" />
+            <origin xyz="0.0 0 0.2" rpy="0 0 0" />
             <geometry>
                <mesh filename="package://niryo_one_description/meshes/v2/stl/G2_Clamp.STL" scale="0.001 0.001 0.001"/>
@@ -294,5 +294,5 @@
          </visual>
          <collision>
-            <origin xyz="0.0 0.0 0.0" rpy="0 0 0" />
+            <origin xyz="0.0 -0.1 0.0" rpy="0 0 0" />
             <geometry>
                <mesh filename="package://niryo_one_description/meshes/v2/stl/G2_Rod.STL" scale="0.001 0.001 0.001"/>
@@ -328,13 +328,20 @@
     </gazebo>
     <!-- hack from here: https://github.com/JenniferBuehler/gazebo-pkgs/wiki/The-Gazebo-grasp-fix-plugin -->
+    <!-- This plugin does not seem to be loaded -->
+    <!-- Also this plugin seems to require all the finger links to be attached
+         to a link (palm link) which in our case does not happen.
+         There are the gear links between the hand link and the finger links -->
     <gazebo>
        <plugin name="gazebo_grasp_fix" filename="libgazebo_grasp_fix.so">
             <arm>
                <arm_name>niryo-arm</arm_name>
-               <palm_link>hand_link</palm_link>
+               <!--palm_link>hand_link</palm_link-->
+               <palm_link>gripper_base_link</palm_link>
+               <gripper_link>${prefix}gear_left_link</gripper_link>
+               <gripper_link>${prefix}gear_right_link</gripper_link>
                <gripper_link>${prefix}left_finger_base_link</gripper_link>
                <gripper_link>${prefix}right_finger_base_link</gripper_link>
             </arm>
-           <forces_angle_tolerance>100</forces_angle_tolerance>
+           <forces_angle_tolerance>10</forces_angle_tolerance> <!-- was 100 -->
            <update_rate>4</update_rate>
            <grip_count_threshold>4</grip_count_threshold>
