Commit message: grasp and realease works. Pysics engine tuning needs some work

File: niryo_one_description/urdf/v2/gripper/niryo_gripper_1.urdf.xacro (robot description, xacro)
@@ -122,7 +122,13 @@
          <axis xyz="-1 0 0" />
          <limit effort="10" lower="-0.015" upper="-0.001" velocity="0.041"/>
+         <dynamics damping="0.7" />
+    		 <dynamics damping="1" friction="1"/>
       </joint>
       <gazebo reference="${prefix}left_finger_joint">
         <implicitSpringDamper>1</implicitSpringDamper>
+    		<!--mu1>10.0</mu1>
+    		<mu2>10.0</mu2>
+    		<fdir1>0 1 0</fdir1>
+    		<minDepth>0.01</minDepth-->
       </gazebo>
       <link name="${prefix}left_finger_link">
@@ -133,5 +139,5 @@
          </inertial>
          <visual>
-            <origin xyz="0.0 0 0" rpy="0 0 0" />
+            <origin xyz="0.0 -0.01 0" rpy="0 0 0" />
             <geometry>
                <mesh filename="package://niryo_one_description/meshes/v2/stl/G1_ClampLeft.STL" scale="0.001 0.001 0.001"/>
@@ -142,8 +148,20 @@
          </visual>
          <collision>
-            <origin xyz="0.0 0 0" rpy="0 0 0" />
+            <origin xyz="0.0 -0.01 0" rpy="0 0 0" />
             <geometry>
                <mesh filename="package://niryo_one_description/meshes/v2/stl/G1_ClampLeft.STL" scale="0.001 0.001 0.001"/>
             </geometry>
+						<!--surface>
+							<friction>
+								<ode>
+									<mu1>1.0</mu1>
+									<mu2>1.0</mu2>
+									<minDepth>0.003</minDepth>
+									<maxVel>0</maxVel>
+									<slip1>0</slip1>
+									<slip2>0</slip2>
+								</ode>
+							</friction>
+						</surface-->
          </collision>
       </link>
@@ -161,14 +179,14 @@
          </inertial>
          <visual>
-            <origin xyz="0.0 0 0" rpy="0 0 0" />
-            <geometry>
-               <mesh filename="package://niryo_one_description/meshes/v2/stl/G1_Rod.STL" scale="0.001 0.001 0.001"/>
-            </geometry>
-            <material name="black">
-  		<color rgba="0.0 0.0 0.0 1.0"/>
-            </material>
-         </visual>
-         <collision>
-            <origin xyz="0.0 0 0" rpy="0 0 0" />
+            <origin xyz="0 0 0" rpy="0 0 0" />
+            <geometry>
+               <mesh filename="package://niryo_one_description/meshes/v2/stl/G1_Rod.STL" scale="0.001 0.001 0.001"/>
+            </geometry>
+            <material name="black">
+  		<color rgba="0.0 0.0 0.0 1.0"/>
+            </material>
+         </visual>
+         <collision>
+            <origin xyz="0 0 0" rpy="0 0 0" />
             <geometry>
                <mesh filename="package://niryo_one_description/meshes/v2/stl/G1_Rod.STL" scale="0.001 0.001 0.001"/>
@@ -181,10 +199,16 @@
          <child link="${prefix}right_finger_link"/>
          <origin xyz="0.003 -0.017 0.019" rpy="3.14 0 3.14" />
-	 <axis xyz="-1 0 0" />
+	       <axis xyz="-1 0 0" />
          <limit effort="10" lower="0.001" upper="0.015" velocity="0.041"/>
+				 <dynamics damping="0.7" />
+    		 <dynamics damping="1" friction="1"/>
       </joint>
       <gazebo reference="${prefix}right_finger_joint">
         <implicitSpringDamper>1</implicitSpringDamper>
-      </gazebo>
+    		<!--mu1>10.0</mu1>
+    		<mu2>10.0</mu2>
+    		<fdir1>0 -1 0</fdir1>
+    		<minDepth>0.01</minDepth-->
+			</gazebo>
       <link name="${prefix}right_finger_link">
          <inertial>
@@ -194,5 +218,5 @@
          </inertial>
          <visual>
-            <origin xyz="0.0 0 0" rpy="0 0 0" />
+            <origin xyz="0 -0.01 0" rpy="0 0 0" />
             <geometry>
                <mesh filename="package://niryo_one_description/meshes/v2/stl/G1_ClampRight.STL" scale="0.001 0.001 0.001"/>
@@ -203,10 +227,23 @@
          </visual>
          <collision>
-            <origin xyz="0.0 0 0" rpy="0 0 0" />
+            <origin xyz="0.0 -0.01 0" rpy="0 0 0" />
             <geometry>
                <mesh filename="package://niryo_one_description/meshes/v2/stl/G1_ClampRight.STL" scale="0.001 0.001 0.001"/>
             </geometry>
-         </collision>
-      </link>
+						<!--surface>
+							<friction>
+								<ode>
+            			<mu1>1.0</mu1>
+  								<mu2>1.0</mu2>
+  								<minDepth>0.003</minDepth>
+  								<maxVel>0</maxVel>
+									<slip1>0</slip1>
+									<slip2>0</slip2>
+								</ode>
+							</friction>
+						</surface-->
+         </collision>
+      </link>
+    <!--
     <gazebo>
     <plugin name='ft_sensor_l' filename='libgazebo_ros_ft_sensor.so'>
@@ -222,9 +259,10 @@
     </plugin>
     </gazebo>
+    -->
     <!-- hack from here: https://github.com/JenniferBuehler/gazebo-pkgs/wiki/The-Gazebo-grasp-fix-plugin -->
     <gazebo>
        <plugin name="gazebo_grasp_fix" filename="libgazebo_grasp_fix.so">
             <arm>
-               <arm_name>niryo-arm</arm_name>
+               <arm_name>/niryo_one</arm_name>
                <palm_link>hand_link</palm_link>
                <gripper_link>${prefix}left_finger_link</gripper_link>
@@ -235,5 +273,5 @@
            <grip_count_threshold>4</grip_count_threshold>
            <max_grip_count>8</max_grip_count>
-           <release_tolerance>0.005</release_tolerance>
+           <release_tolerance>0.001</release_tolerance>
            <disable_collisions_on_attach>false</disable_collisions_on_attach>
            <contact_topic>__default_topic__</contact_topic>

File: niryo_one_description/urdf/v2/gripper/niryo_gripper_2.urdf.xacro (robot description, xacro)
@@ -9,6 +9,10 @@
       <inertia ixx="${m*(3*r*r+h*h)/12}" ixy = "0" ixz = "0" iyy="${m*(3*r*r+h*h)/12}" iyz = "0" izz="${m*r*r/2}" />
    </xacro:macro>
-    <!-- The gripper needs to be fixed -->
-    <!-- Should add gripper and transmission tags to gripper joints -->
+   <xacro:macro name="default_origin">
+     <origin xyz="0 0 0" rpy="0 0 0"/>
+		 </xacro:macro>
+	 <xacro:default_origin />
+   <!-- The gripper needs to be fixed -->
+   <!-- Should add gripper and transmission tags to gripper joints -->
    <xacro:macro name="default_transmission" params="jname">
     <transmission name="${jname}_trans">
@@ -33,5 +37,5 @@
       <link name="${prefix}base_link">
          <inertial>
-            <mass value="0.25" />
+            <mass value="0.20" />
             <origin xyz="0 0 0" />
             <cylinder_inertia m="0.20" r="0.05" h="0.05" />
@@ -62,5 +66,5 @@
          <parent link="${prefix}base_link"/>
          <child link="${prefix}gear_left_link"/>
-            <origin xyz="0.016 0.0 0.005" rpy="0 0 0" />
+            <origin xyz="0.018 0.0 0.005" rpy="0 0 0" />
          <axis xyz="0 -1 0" />
  	       <limit effort="1000.0" lower="-1.2" upper="0.0" velocity="0.5"/>
@@ -72,11 +76,11 @@
       <link name="${prefix}gear_left_link">
          <inertial>
-            <mass value="0.25" />
-            <origin xyz="0 0 0" />
-            <cylinder_inertia m="0.20" r="0.05" h="0.05" />
-            <gravity>1</gravity>
-         </inertial>
-         <visual>
-         <origin xyz="-0.025 0.02 0.045" rpy="3.14 0.0 0.0" />
+            <mass value="0.20" />
+            <origin xyz="0 0 0" />
+            <cylinder_inertia m="0.20" r="0.05" h="0.05" />
+            <gravity>1</gravity>
+         </inertial>
+         <visual>
+            <origin xyz="-0.025 0.02 0.045" rpy="3.14 0 0" />
             <geometry>
                <mesh filename="package://niryo_one_description/meshes/v2/stl/G2_GearLeft.STL" scale="0.001 0.001 0.001"/>
@@ -87,5 +91,5 @@
          </visual>
          <collision>
-            <origin xyz="0.0 0 0" rpy="0 0 0" />
+            <origin xyz="-0.025 0.02 0.045" rpy="3.14 0 0" />
             <geometry>
                <mesh filename="package://niryo_one_description/meshes/v2/stl/G2_GearLeft.STL" scale="0.001 0.001 0.001"/>
@@ -97,5 +101,5 @@
          <parent link="${prefix}base_link"/>
          <child link="${prefix}gear_right_link"/>
-         <origin xyz="-0.003 0 0.005" rpy="0 0.0 0.0" />
+         <origin xyz="-0.005 0 0.005" rpy="0 0.0 0.0" />
       <axis xyz="0 -1 0" />
  	 <limit effort="1000.0" lower="0" upper="1.2" velocity="0.5"/>
@@ -107,11 +111,11 @@
       <link name="${prefix}gear_right_link">
          <inertial>
-            <mass value="0.25" />
-            <origin xyz="0 0 0" />
-            <cylinder_inertia m="0.20" r="0.05" h="0.05" />
-            <gravity>1</gravity>
-         </inertial>
-         <visual>
-            <origin xyz="-0.008 0.02 0.045" rpy="3.14 0  0" />
+            <mass value="0.20" />
+            <origin xyz="0 0 0" />
+            <cylinder_inertia m="0.20" r="0.05" h="0.05" />
+            <gravity>1</gravity>
+         </inertial>
+         <visual>
+            <origin xyz="-0.008 0.02 0.045" rpy="3.14 0 0" />
             <geometry>
                <mesh filename="package://niryo_one_description/meshes/v2/stl/G2_GearRight.STL" scale="0.001 0.001 0.001"/>
@@ -122,5 +126,5 @@
          </visual>
          <collision>
-            <origin xyz="0.0 0.0 0.0" rpy="0 0 0" />
+            <origin xyz="-0.008 0.02 0.045" rpy="3.14 0 0" />
             <geometry>
                <mesh filename="package://niryo_one_description/meshes/v2/stl/G2_GearRight.STL" scale="0.001 0.001 0.001"/>
@@ -142,5 +146,5 @@
           <gazebo/>
         </limit>
-	      <mimic joint="${prefix}gear_left_joint" multiplier="-1" offset="0"/>
+	      <!--mimic joint="${prefix}gear_left_joint" multiplier="-1" offset="0"/-->
       </joint>
       <gazebo reference="${prefix}left_finger_base_joint">
@@ -165,8 +169,16 @@
          </visual>
          <collision>
-            <origin xyz="0.0 0.0 0.2" rpy="0 0 0" />
+            <origin xyz="-0.001 -0.007 0.011" rpy="0 3.14 0" />
             <geometry>
                <mesh filename="package://niryo_one_description/meshes/v2/stl/G2_Clamp.STL" scale="0.001 0.001 0.001"/>
             </geometry>
+            <surface>
+              <friction>
+                <ode>
+                  <mu>0.8</mu>
+                  <mu2>0.8</mu2>
+                </ode>
+              </friction>
+            </surface>
          </collision>
       </link>
@@ -185,5 +197,5 @@
           <gazebo/>
         </limit>
-	      <mimic joint="${prefix}gear_right_joint" multiplier="-1" offset="0"/>
+	      <!--mimic joint="${prefix}gear_right_joint" multiplier="-1" offset="0"/-->
       </joint>
       <gazebo reference="${prefix}right_finger_base_joint">
@@ -208,8 +220,16 @@
          </visual>
          <collision>
-            <origin xyz="0.0 0 0.2" rpy="0 0 0" />
+            <origin xyz="0.002 0.02 0.011" rpy="0 3.14 3.14" />
             <geometry>
                <mesh filename="package://niryo_one_description/meshes/v2/stl/G2_Clamp.STL" scale="0.001 0.001 0.001"/>
             </geometry>
+            <surface>
+              <friction>
+              <ode>
+                <mu>0.8</mu>
+                <mu2>0.8</mu2>
+              </ode>
+            </friction>
+            </surface>
          </collision>
       </link>
@@ -228,5 +248,5 @@
           <gazebo/>
         </limit>
-	      <mimic joint="${prefix}gear_left_joint" multiplier="1" offset="0"/>
+	      <!--mimic joint="${prefix}gear_left_joint" multiplier="1" offset="0"/-->
       </joint>
        <gazebo reference="${prefix}rod_left_joint">
@@ -236,11 +256,11 @@
       <link name="${prefix}rod_left_link">
          <inertial>
-            <mass value="0.25" />
-            <origin xyz="0 0 0" />
-            <cylinder_inertia m="0.20" r="0.05" h="0.05" />
-            <gravity>1</gravity>
-         </inertial>
-         <visual>
-	<origin xyz="0.027 0.02 0.008" rpy="0.0 0.0 3.14" />
+            <mass value="0.20" />
+            <origin xyz="0 0 0" />
+            <cylinder_inertia m="0.20" r="0.05" h="0.05" />
+            <gravity>1</gravity>
+         </inertial>
+         <visual>
+            <origin xyz="0.027 0.02 0.008" rpy="0 0 3.14" />
             <geometry>
                <mesh filename="package://niryo_one_description/meshes/v2/stl/G2_Rod.STL" scale="0.001 0.001 0.001"/>
@@ -251,5 +271,5 @@
          </visual>
          <collision>
-            <origin xyz="0.0 0.0 0.0" rpy="0 0 0" />
+            <origin xyz="0.027 0.02 0.008" rpy="0 0 3.14" />
             <geometry>
                <mesh filename="package://niryo_one_description/meshes/v2/stl/G2_Rod.STL" scale="0.001 0.001 0.001"/>
@@ -271,5 +291,5 @@
           <gazebo/>
         </limit>
-	      <mimic joint="${prefix}gear_right_joint" multiplier="1" offset="0.0"/>
+	      <!--mimic joint="${prefix}gear_right_joint" multiplier="1" offset="0.0"/-->
       </joint>
       <gazebo reference="${prefix}rod_right_joint">
@@ -285,5 +305,5 @@
          </inertial>
          <visual>
-	<origin xyz="-0.027 -0.007 0.008" rpy="0.0 0.0 0.0" />
+            <origin xyz="-0.027 -0.007 0.008" rpy="0 0 0" />
             <geometry>
                <mesh filename="package://niryo_one_description/meshes/v2/stl/G2_Rod.STL" scale="0.001 0.001 0.001"/>
@@ -294,5 +314,5 @@
          </visual>
          <collision>
-            <origin xyz="0.0 -0.1 0.0" rpy="0 0 0" />
+            <origin xyz="-0.027 -0.007 0.008" rpy="0 0 0" />
             <geometry>
                <mesh filename="package://niryo_one_description/meshes/v2/stl/G2_Rod.STL" scale="0.001 0.001 0.001"/>
@@ -328,20 +348,19 @@
     </gazebo>
     <!-- hack from here: https://github.com/JenniferBuehler/gazebo-pkgs/wiki/The-Gazebo-grasp-fix-plugin -->
-    <!-- This plugin does not seem to be loaded -->
+    <!-- This plugin seems to be loaded -->
     <!-- Also this plugin seems to require all the finger links to be attached
          to a link (palm link) which in our case does not happen.
-         There are the gear links between the hand link and the finger links -->
+There are the gear links between the hand link and the finger links -->
     <gazebo>
        <plugin name="gazebo_grasp_fix" filename="libgazebo_grasp_fix.so">
             <arm>
-               <arm_name>niryo-arm</arm_name>
+               <arm_name>/niryo_one</arm_name>
                <!--palm_link>hand_link</palm_link-->
-               <palm_link>gripper_base_link</palm_link>
-               <gripper_link>${prefix}gear_left_link</gripper_link>
-               <gripper_link>${prefix}gear_right_link</gripper_link>
+               <!--gripper_link>${prefix}gear_right_link</gripper_link-->
+               <palm_link>${prefix}gear_left_link</palm_link>
                <gripper_link>${prefix}left_finger_base_link</gripper_link>
                <gripper_link>${prefix}right_finger_base_link</gripper_link>
             </arm>
-           <forces_angle_tolerance>10</forces_angle_tolerance> <!-- was 100 -->
+           <forces_angle_tolerance>100</forces_angle_tolerance>
            <update_rate>4</update_rate>
            <grip_count_threshold>4</grip_count_threshold>
@@ -354,4 +373,8 @@
     <xacro:default_transmission jname="${prefix}gear_left"/>
     <xacro:default_transmission jname="${prefix}gear_right"/>
+    <xacro:default_transmission jname="${prefix}rod_left"/>
+    <xacro:default_transmission jname="${prefix}rod_right"/>
+    <xacro:default_transmission jname="${prefix}left_finger_base"/>
+    <xacro:default_transmission jname="${prefix}right_finger_base"/>
    </xacro:macro>
 </robot>

File: niryo_one_description/urdf/v2/niryo_one.urdf (robot description, URDF)
Before this commit: robot niryo_one, 16 links, 15 joints
Links:
- removed link gripper_rod_right_link
- added link gripper_rod_right_link_george, mass 0.25; collision mesh filename=package://niryo_one_description/meshes/v2/stl/G2_Rod.STL scale=0.001 0.001 0.001; visual mesh filename=package://niryo_one_description/meshes/v2/stl/G2_Rod.STL scale=0.001 0.001 0.001
Joints:
- joint gripper_left_finger_base_joint: mimic joint=gripper_gear_left_joint multiplier=-1 offset=0 -> (none)
- joint gripper_right_finger_base_joint: mimic joint=gripper_gear_right_joint multiplier=-1 offset=0 -> (none)
- joint gripper_rod_left_joint: mimic joint=gripper_gear_left_joint multiplier=1 offset=0 -> (none)
- joint gripper_rod_right_joint: mimic joint=gripper_gear_right_joint multiplier=1 offset=0.0 -> (none)

File: niryo_one_description/urdf/v2/niryo_one.urdf.xacro (robot description, xacro)
@@ -44,6 +44,6 @@
 	<xacro:include filename="$(find niryo_one_description)/urdf/gazebo/niryo_one.transmission.xacro" />
 	<!-- Gripper -->
-<!--	<xacro:include filename="$(find niryo_one_description)/urdf/v2/gripper/niryo_gripper_1.urdf.xacro" />  -->
-	<xacro:include filename="$(find niryo_one_description)/urdf/v2/gripper/niryo_gripper_2.urdf.xacro" />
+	<xacro:include filename="$(find niryo_one_description)/urdf/v2/gripper/niryo_gripper_1.urdf.xacro" />
+	<!--xacro:include filename="$(find niryo_one_description)/urdf/v2/gripper/niryo_gripper_2.urdf.xacro" /-->
 	<!-- Links -->
     <link name="ground_link"/>
@@ -264,14 +264,16 @@
         <origin xyz="0 0 ${distance_hand_tool}" rpy="${-PI/2} ${-PI/2} 0" />
 	</joint>
-<!--	<xacro:niryo_gripper_1 prefix="gripper_" parent="tool_link" >
+	<xacro:niryo_gripper_1 prefix="gripper_" parent="tool_link" >
 	  <origin xyz="0.025 0 -0.013" rpy="${PI/2} ${PI} ${PI/2} " />
 	</xacro:niryo_gripper_1>
--->
-	<xacro:niryo_gripper_2 prefix="gripper_" parent="tool_link" >
+	<!--xacro:niryo_gripper_2 prefix="gripper_" parent="tool_link" >
 	  <origin xyz="0.025 0 -0.013" rpy="${PI/2} ${PI} ${PI/2} " />
-	</xacro:niryo_gripper_2>
+	</xacro:niryo_gripper_2-->
     <!--plugin-->
 	<gazebo>
   		<plugin name="gazebo_ros_control" filename="libgazebo_ros_control.so">
+      	<robotNamespace></robotNamespace>
+    		<robotSimType>gazebo_ros_control/DefaultRobotHWSim</robotSimType>
+    		<legacyModeNS>true</legacyModeNS>
   		</plugin>
   	</gazebo>
